Commit message: fix joints names

File: src/rovi_description/urdf/rovi.urdf (robot description, URDF)
Before this commit: robot rovi, 8 links, 7 joints
Joints:
- removed joint front_left_wheel_joint
- removed joint front_right_wheel_joint
- added joint front_left_joint: type continuous, parent base_link, child front_left_wheel, origin xyz=0.08 0.084492 -0.0389 rpy=1.57079632679 0 0, axis 0 0 1, limit lower=-3.14159265359 upper=3.14159265359 effort=100 velocity=1
- added joint front_right_joint: type continuous, parent base_link, child front_right_wheel, origin xyz=0.08 -0.0845 -0.0389 rpy=-1.57079632679 0 3.14159265359, axis 0 0 1, limit lower=-3.14159265359 upper=3.14159265359 effort=100 velocity=1

Commit message: adjusted robot mesh to correct model

File: src/rovi_description/urdf/rovi.urdf (robot description, URDF)
Before this commit: robot rovi, 8 links, 7 joints
Links:
- link back_left_wheel: geometry collision mesh filename=package://rovi_description/meshes/mecanum/wheel_RL_FR.stl; visual mesh filename=package://rovi_description/meshes/mecanum/wheel_RL_FR.stl
- link back_right_wheel: geometry collision mesh filename=package://rovi_description/meshes/mecanum/wheel_RR_FL.stl; visual mesh filename=package://rovi_description/meshes/mecanum/wheel_RR_FL.stl
- link base_link: geometry collision mesh filename=package://rovi_description/meshes/mecanum/chassis.stl; visual mesh filename=package://rovi_description/meshes/mecanum/chassis.stl
- link front_left_wheel: geometry collision mesh filename=package://rovi_description/meshes/mecanum/wheel_RR_FL.stl; visual mesh filename=package://rovi_description/meshes/mecanum/wheel_RR_FL.stl
- link front_right_wheel: geometry collision mesh filename=package://rovi_description/meshes/mecanum/wheel_RL_FR.stl; visual mesh filename=package://rovi_description/meshes/mecanum/wheel_RL_FR.stl
Joints:
- joint back_left_joint: origin xyz=-0.08 0.084492 -0.03954 rpy=1.57079632679 0 0 -> xyz=-0.08231 0.1041 0.0135 rpy=1.57079632679 0 0
- joint back_right_joint: origin xyz=-0.08 -0.0845 -0.03946 rpy=-1.57079632679 0 3.14159265359 -> xyz=-0.080231 -0.1041 0.0135 rpy=-1.57079632679 0 3.14159265359
- joint base_joint: origin xyz=0.0 0.0 0.0815 rpy=0 0 0 -> xyz=0.0 0.0 0.029 rpy=0 0 0
- joint front_left_joint: origin xyz=0.08 0.084492 -0.0389 rpy=1.57079632679 0 0 -> xyz=0.139 0.10406 0.0139 rpy=1.57079632679 0 0
- joint front_right_joint: origin xyz=0.08 -0.0845 -0.0389 rpy=-1.57079632679 0 3.14159265359 -> xyz=0.13902 -0.10414 0.010269 rpy=-1.57079632679 0 3.14159265359

Commit message: fixed laser joint position

File: src/rovi_description/urdf/rovi.urdf (robot description, URDF)
Before this commit: robot rovi, 8 links, 7 joints
Joints:
- joint laser_joint: origin xyz=0 0 0.15 rpy=0 0 0 -> xyz=0.129 0 0.1645 rpy=0 0 0

Commit message: fix lidar signal rotation

File: src/rovi_description/urdf/rovi.urdf (robot description, URDF)
Before this commit: robot rovi, 8 links, 7 joints
Joints:
- joint laser_joint: origin xyz=0.129 0 0.1645 rpy=0 0 0 -> xyz=0.129 0 0.1645 rpy=0 0 3.14159

Commit message: fix URDF rotation already compensated in driver

File: src/rovi_description/urdf/rovi.urdf (robot description, URDF)
Before this commit: robot rovi, 8 links, 7 joints
Joints:
- joint base_imu: origin xyz=-0.06 0.01 0.01 rpy=0 3.1415 1.5707 -> xyz=0.06 0.03 0.01 rpy=0 0 0

Commit message: urdf collision

File: src/rovi_description/urdf/rovi.urdf (robot description, URDF)
Before this commit: robot rovi, 8 links, 7 joints
Links:
- link back_left_wheel: geometry collision cylinder length=0.037 radius=0.04; visual mesh filename=package://rovi_description/meshes/mecanum/wheel_RL_FR.stl
- link back_right_wheel: geometry collision cylinder length=0.037 radius=0.04; visual mesh filename=package://rovi_description/meshes/mecanum/wheel_RR_FL.stl
- link front_left_wheel: geometry collision cylinder length=0.037 radius=0.04; visual mesh filename=package://rovi_description/meshes/mecanum/wheel_RR_FL.stl
- link front_right_wheel: geometry collision cylinder length=0.037 radius=0.04; visual mesh filename=package://rovi_description/meshes/mecanum/wheel_RL_FR.stl

Commit message: added depth camera in sim

File: src/rovi_description/urdf/rovi.urdf (robot description, URDF)
Before this commit: robot rovi, 8 links, 7 joints
Links:
- added link camera_color_frame
- added link camera_color_optical_frame
- added link camera_depth_frame
- added link camera_depth_optical_frame
- added link camera_link
Joints:
- added joint camera_color_optical_joint: type fixed, parent camera_color_frame, child camera_color_optical_frame, origin xyz=0 0 0 rpy=-1.57079632679 0 -1.57079632679
- added joint camera_depth_optical_joint: type fixed, parent camera_depth_frame, child camera_depth_optical_frame, origin xyz=0 0 0 rpy=-1.57079632679 0 -1.57079632679
- added joint camera_joint: type fixed, parent base_link, child camera_link, origin xyz=0.129 0 0.10 rpy=0 0 0
- added joint camera_link_to_depth_frame: type fixed, parent camera_link, child camera_depth_frame, origin xyz=0 -0.02 0 rpy=0 0 0
- added joint camera_link_to_rgb_frame: type fixed, parent camera_link, child camera_color_frame, origin xyz=0 -0.045 0 rpy=0 0 0

Commit message: plan for known floor geometry

File: src/rovi_description/urdf/rovi.urdf (robot description, URDF)
Before this commit: robot rovi, 13 links, 12 joints
Joints:
- joint camera_joint: origin xyz=0.129 0 0.10 rpy=0 0 0 -> xyz=0.129 0 0.086 rpy=0 0 0
